File: Tiny85_SP_Breakout.kicad_pcb (KiCad board)
At the start: 2 copper layers, 14.9 x 8.4 mm, 5 parts, among them J1 Conn_01x02_Female, J2 Conn_01x04_Female, J3 Conn_01x02_Female, U1 ATtiny85-20SU

Commit message: Update to v2
Parts:
- moved J3 0.34 mm to (159.8, 100.2)
- moved C1 0.14 mm to (157.1, 97.2)
Other:
- board size 14.9 x 8.4 mm -> 15.2 x 8.4 mm
- board text added: "+"
- board text added: "5/rst"
- board text added: "ATtiny85"
- board text added: "int"
- board text added: "⏚"
- board text removed: "G"
- board text removed: "V"
Changed lines of the file:
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@@
   (general
     (thickness 1.6)
-    (drawings 22)
+    (drawings 43)
     (tracks 45)
     (zones 0)
@@
   (page A4)
   (layers
-    (0 F.Cu signal hide)
-    (31 B.Cu signal hide)
+    (0 F.Cu signal)
+    (31 B.Cu signal)
     (32 B.Adhes user)
     (33 F.Adhes user)
@@
     (37 F.SilkS user)
     (38 B.Mask user)
-    (39 F.Mask user hide)
+    (39 F.Mask user)
     (40 Dwgs.User user)
     (41 Cmts.User user)
@@
   )
   (module Capacitor_SMD:C_0603_1608Metric_Pad1.05x0.95mm_HandSolder (layer F.Cu)
-    (at 157.125 97.318718 180)
+    (at 157.115 97.18 180)
     (descr "Capacitor SMD 0603 (1608 Metric), square (rectangular) end terminal, IPC_7351 nominal with elongated pad for handsoldering. (Body size source: http://www.tortai-tech.com/upload/download/2011102023233369053.pdf), generated with kicad-footprint-generator")
     (tags "capacitor handsolder")
@@
   )
   (module Connector:2_tiny_pads (layer F.Cu)
-    (at 160.14 100.33 270)
+    (at 159.84 100.17 270)
     (fp_text reference J3 (at 0 0.5 90) (layer F.SilkS) hide
       (effects (font (size 1 1) (thickness 0.15)))
@@
     )
   )
+  (gr_text ATtiny85 (at 151.45 99.25) (layer F.SilkS)
+    (effects (font (size 0.7 0.7) (thickness 0.1)))
+  )
+  (gr_text int (at 145.575 96.8) (layer F.SilkS)
+    (effects (font (size 0.6 0.6) (thickness 0.1)))
+  )
+  (gr_line (start 144.5 102.126556) (end 145.775 102.475) (layer F.SilkS) (width 0.12))
+  (gr_line (start 144.5 102.368845) (end 145.775 102.025) (layer F.SilkS) (width 0.12))
+  (gr_circle (center 144.5 102.575) (end 144.55 102.375) (layer F.SilkS) (width 0.12))
+  (gr_circle (center 144.5 101.925) (end 144.6 102.1) (layer F.SilkS) (width 0.12))
+  (gr_text 5/rst (at 157.275 103.75) (layer F.SilkS)
+    (effects (font (size 0.6 0.6) (thickness 0.1)))
+  )
+  (gr_text 4 (at 153.7 103.775) (layer F.SilkS)
+    (effects (font (size 0.6 0.6) (thickness 0.1)))
+  )
+  (gr_text 1 (at 149.125 103.775) (layer F.SilkS)
+    (effects (font (size 0.6 0.6) (thickness 0.1)))
+  )
+  (gr_text 0 (at 146.525 103.8) (layer F.SilkS)
+    (effects (font (size 0.6 0.6) (thickness 0.1)))
+  )
+  (gr_text 2 (at 144.325 98.225) (layer F.SilkS)
+    (effects (font (size 0.6 0.6) (thickness 0.1)))
+  )
+  (gr_text + (at 144.325 100.775) (layer F.SilkS)
+    (effects (font (size 0.7 0.7) (thickness 0.1)))
+  )
+  (gr_text 3 (at 158.6 101.5) (layer F.SilkS)
+    (effects (font (size 0.6 0.6) (thickness 0.1)))
+  )
+  (gr_text ⏚ (at 158.625 98.85) (layer F.SilkS)
+    (effects (font (size 0.7 0.7) (thickness 0.1)))
+  )
+  (gr_line (start 157.91 102.25) (end 158.95 102.25) (layer F.SilkS) (width 0.08))
+  (gr_line (start 155.95 102.25) (end 156.99 102.25) (layer F.SilkS) (width 0.08))
+  (gr_line (start 153.81 102.25) (end 154.85 102.25) (layer F.SilkS) (width 0.08))
+  (gr_line (start 151.81 102.25) (end 152.85 102.25) (layer F.SilkS) (width 0.08))
+  (gr_line (start 149.785 102.25) (end 150.825 102.25) (layer F.SilkS) (width 0.08))
+  (gr_line (start 147.835 102.25) (end 148.875 102.25) (layer F.SilkS) (width 0.08))
+  (gr_line (start 146.025 102.25) (end 147.065 102.25) (layer F.SilkS) (width 0.08))
+  (gr_text ⏚ (at 157.3 98.95) (layer B.SilkS)
+    (effects (font (size 1 1) (thickness 0.15)) (justify mirror))
+  )
   (gr_text "… or do, I’m a\npcb, not a cop" (at 151.6 99.9) (layer B.SilkS)
     (effects (font (size 0.65 0.65) (thickness 0.15)) (justify mirror))
@@
   )
   (gr_circle (center 147.6 103.1) (end 146.8 102.7) (layer B.SilkS) (width 0.12))
-  (gr_circle (center 150.2 103.1) (end 149.4 102.7) (layer B.SilkS) (width 0.12))
-  (gr_circle (center 152.7 103.1) (end 151.9 102.7) (layer B.SilkS) (width 0.12))
-  (gr_circle (center 155.2 103.1) (end 154.4 102.7) (layer B.SilkS) (width 0.12))
-  (gr_circle (center 157.6 101.5) (end 156.8 101.1) (layer B.SilkS) (width 0.12))
-  (gr_circle (center 157.6 99) (end 156.8 98.6) (layer B.SilkS) (width 0.12))
+  (gr_circle (center 150.155573 103.1) (end 149.355573 102.7) (layer B.SilkS) (width 0.12))
+  (gr_circle (center 152.669427 103.1) (end 151.869427 102.7) (layer B.SilkS) (width 0.12))
+  (gr_circle (center 155.219427 103.1) (end 154.419427 102.7) (layer B.SilkS) (width 0.12))
+  (gr_circle (center 157.32 101.344427) (end 156.52 100.944427) (layer B.SilkS) (width 0.12))
+  (gr_circle (center 157.3 98.89) (end 156.5 98.49) (layer B.SilkS) (width 0.12))
   (gr_circle (center 145.6 98.2) (end 144.8 97.8) (layer B.SilkS) (width 0.12))
-  (gr_circle (center 145.6 100.7) (end 144.8 100.3) (layer B.SilkS) (width 0.12))
+  (gr_circle (center 145.6 100.755573) (end 144.8 100.355573) (layer B.SilkS) (width 0.12))
   (gr_text 5 (at 155.2 103.2) (layer B.SilkS)
     (effects (font (size 1 1) (thickness 0.15)) (justify mirror))
@@
     (effects (font (size 1 1) (thickness 0.15)) (justify mirror))
   )
-  (gr_text 3 (at 157.6 101.6) (layer B.SilkS)
-    (effects (font (size 1 1) (thickness 0.15)) (justify mirror))
-  )
-  (gr_text G (at 157.7 99.1) (layer B.SilkS)
+  (gr_text 3 (at 157.275 101.425) (layer B.SilkS)
     (effects (font (size 1 1) (thickness 0.15)) (justify mirror))
   )
@@
     (effects (font (size 1 1) (thickness 0.15)) (justify mirror))
   )
-  (gr_text V (at 145.6 100.9) (layer B.SilkS)
+  (gr_text + (at 145.59 100.66) (layer B.SilkS)
     (effects (font (size 1 1) (thickness 0.15)) (justify mirror))
   )
   (gr_line (start 159.1 95.9) (end 159.1 104.3) (layer Edge.Cuts) (width 0.1))
-  (gr_line (start 144.2 95.9) (end 159.1 95.9) (layer Edge.Cuts) (width 0.1))
-  (gr_line (start 144.2 104.3) (end 144.2 95.9) (layer Edge.Cuts) (width 0.1))
-  (gr_line (start 159.1 104.3) (end 144.2 104.3) (layer Edge.Cuts) (width 0.1))
+  (gr_line (start 143.875 95.875) (end 159.1 95.9) (layer Edge.Cuts) (width 0.1))
+  (gr_line (start 143.875 104.3) (end 143.875 95.875) (layer Edge.Cuts) (width 0.1))
+  (gr_line (start 159.1 104.3) (end 143.875 104.3) (layer Edge.Cuts) (width 0.1))
   (segment (start 147.385 100.74) (end 147.774999 101.129999) (width 0.25) (layer F.Cu) (net 1))
   (segment (start 145.6 100.74) (end 147.385 100.74) (width 0.25) (layer F.Cu) (net 1))
@@
   (segment (start 155.22 101.275) (end 155.074999 101.129999) (width 0.25) (layer F.Cu) (net 7))
   (segment (start 155.22 103) (end 155.22 101.275) (width 0.25) (layer F.Cu) (net 7))
-  (segment (start 157.6 101.285) (end 157.6 101.6) (width 0.25) (layer F.Cu) (net 8))
+  (segment (start 157.35 101.285) (end 157.35 101.6) (width 0.25) (layer F.Cu) (net 8))
   (segment (start 156.174999 99.859999) (end 157.6 101.285) (width 0.25) (layer F.Cu) (net 8))
   (segment (start 155.074999 99.859999) (end 156.174999 99.859999) (width 0.25) (layer F.Cu) (net 8))
